File: hardware/kicad/bwlr1e.kicad_pcb (KiCad board)
At the start: 2 copper layers, 36.8 x 90.9 mm, 65 parts, among them J1 Qwiic, Q1 AO3407, Q2 DMG1012UW, SW3 RESET, SW4 BOOT, U1 BME688, U2 RAK3172, U3 AEM10941-QFN, U4 XC6215

Commit message: add qwiic silkscreen info
Other:
- board text added: "3V3"
- board text added: "GND"
- board text added: "SCL"
- board text added: "SDA"
Changed lines of the file:
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@@
         (effects (font (size 1 1) (thickness 0.15)) (justify mirror))
     )
-    (fp_text value "Qwiic" (at -6.326 0.603 90) (layer "B.SilkS")
+    (fp_text value "Qwiic" (at -5.818 0.095 90) (layer "B.SilkS")
         (effects (font (size 1 1) (thickness 0.15)) (justify mirror))
     )
@@
     )
   )
+  (gr_text "3V3" (at 136.144 87.122) (layer "B.SilkS")
+    (effects (font (size 0.5 0.5) (thickness 0.125)) (justify left bottom mirror))
+  )
+  (gr_text "SDA" (at 136.144 86.106) (layer "B.SilkS")
+    (effects (font (size 0.5 0.5) (thickness 0.125)) (justify left bottom mirror))
+  )
   (gr_text "Revision 4" (at 161.925 142.367) (layer "B.SilkS" knockout)
     (effects (font (size 0.8 0.8) (thickness 0.2) bold) (justify left bottom mirror))
+  )
+  (gr_text "GND" (at 136.271 88.138) (layer "B.SilkS")
+    (effects (font (size 0.5 0.5) (thickness 0.125)) (justify left bottom mirror))
   )
   (gr_text "BWLR1E" (at 139.065 140.97) (layer "B.SilkS")
@@
     )
   )
+  (gr_text "SCL" (at 136.144 85.09) (layer "B.SilkS")
+    (effects (font (size 0.5 0.5) (thickness 0.125)) (justify left bottom mirror))
+  )
   (gr_text "-" (at 160.16 139.065) (layer "B.SilkS")
