File: hardware/kicad/programmer/bwlr1e-prog.kicad_pcb (KiCad board)
At the start: 2 copper layers, 36.8 x 90.9 mm, 49 parts, among them J1 DEBUG, J2 USB_C_Receptacle_USB2.0, J3 RESET, J4 BOOT, Q1 AO3407A, SW1 SW_DIP_x04, SW4 BOOT, SW5 RESET, U1 USBLC6-2P6, U6 CH340E, U7 MCP73831T-2ACI/OT, U8 XC6220B331MR-G

Commit message: fix filter cap footprint
Parts:
- C2, C4: footprint Capacitor_Tantalum_SMD:CP_EIA-3528-15_AVX-H_Pad1.50x2.35mm_HandSolder -> Capacitor_Tantalum_SMD:CP_EIA-3528-15_AVX-H
Changed lines of the file:
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@@
     )
   )
-  (footprint "Capacitor_Tantalum_SMD:CP_EIA-3528-15_AVX-H_Pad1.50x2.35mm_HandSolder" (layer "F.Cu")
+  (footprint "Capacitor_Tantalum_SMD:CP_EIA-3528-15_AVX-H" (layer "F.Cu")
     (at 158.5462 128.5974)
     (descr "Tantalum Capacitor SMD AVX-H (3528-15 Metric), IPC_7351 nominal, (Body size from: http://www.kemet.com/Lists/ProductCatalog/Attachments/253/KEM_TC101_STD.pdf), generated with kicad-footprint-generator")
@@
     (property "ki_keywords" "cap capacitor")
     (attr smd)
-    (fp_text reference "C2" (at 3.1375 -1.2974) (layer "F.Fab")
-        (effects (font (size 0.5 0.5) (thickness 0.125)))
+    (fp_text reference "C2" (at 0 0.0026) (layer "F.Fab")
+        (effects (font (size 1 1) (thickness 0.15)))
     )
-    (fp_text value "330u" (at 3.1038 0.7026 90) (layer "F.Fab")
-        (effects (font (size 0.5 0.5) (thickness 0.125)))
+    (fp_text value "330u" (at 2.7538 0.0026 90) (layer "F.Fab")
+        (effects (font (size 1 1) (thickness 0.15)))
     )
     (fp_text user "${REFERENCE}" (at 0 0) (layer "F.Fab")
         (effects (font (size 0.88 0.88) (thickness 0.13)))
     )
-    (fp_line (start -2.635 -1.51) (end -2.635 1.51)
+    (fp_line (start -2.46 -1.51) (end -2.46 1.51)
       (stroke (width 0.12) (type solid)) (layer "F.SilkS"))
-    (fp_line (start -2.635 1.51) (end 1.75 1.51)
+    (fp_line (start -2.46 1.51) (end 1.75 1.51)
       (stroke (width 0.12) (type solid)) (layer "F.SilkS"))
-    (fp_line (start 1.75 -1.51) (end -2.635 -1.51)
+    (fp_line (start 1.75 -1.51) (end -2.46 -1.51)
       (stroke (width 0.12) (type solid)) (layer "F.SilkS"))
-    (fp_line (start -2.62 -1.65) (end 2.62 -1.65)
+    (fp_line (start -2.45 -1.65) (end 2.45 -1.65)
       (stroke (width 0.05) (type solid)) (layer "F.CrtYd"))
-    (fp_line (start -2.62 1.65) (end -2.62 -1.65)
+    (fp_line (start -2.45 1.65) (end -2.45 -1.65)
       (stroke (width 0.05) (type solid)) (layer "F.CrtYd"))
-    (fp_line (start 2.62 -1.65) (end 2.62 1.65)
+    (fp_line (start 2.45 -1.65) (end 2.45 1.65)
       (stroke (width 0.05) (type solid)) (layer "F.CrtYd"))
-    (fp_line (start 2.62 1.65) (end -2.62 1.65)
+    (fp_line (start 2.45 1.65) (end -2.45 1.65)
       (stroke (width 0.05) (type solid)) (layer "F.CrtYd"))
     (fp_line (start -1.75 -0.7) (end -1.75 1.4)
@@
     (fp_line (start 1.75 1.4) (end 1.75 -1.4)
       (stroke (width 0.1) (type solid)) (layer "F.Fab"))
-    (pad "1" smd roundrect (at -1.625 0) (size 1.5 2.35) (layers "F.Cu" "F.Paste" "F.Mask") (roundrect_rratio 0.1666673333)
+    (pad "1" smd roundrect (at -1.5375 0) (size 1.325 2.35) (layers "F.Cu" "F.Paste" "F.Mask") (roundrect_rratio 0.188679)
       (net 9 "Net-(BT1-+)") (pintype "passive"))
-    (pad "2" smd roundrect (at 1.625 0) (size 1.5 2.35) (layers "F.Cu" "F.Paste" "F.Mask") (roundrect_rratio 0.1666673333)
+    (pad "2" smd roundrect (at 1.5375 0) (size 1.325 2.35) (layers "F.Cu" "F.Paste" "F.Mask") (roundrect_rratio 0.188679)
       (net 1 "GND") (pintype "passive"))
     (model "${KICAD6_3DMODEL_DIR}/Capacitor_Tantalum_SMD.3dshapes/CP_EIA-3528-15_AVX-H.wrl"
@@
     )
   )
-  (footprint "Capacitor_Tantalum_SMD:CP_EIA-3528-15_AVX-H_Pad1.50x2.35mm_HandSolder" (layer "F.Cu")
+  (footprint "Capacitor_Tantalum_SMD:CP_EIA-3528-15_AVX-H" (layer "F.Cu")
     (at 158.5462 132.2974)
     (descr "Tantalum Capacitor SMD AVX-H (3528-15 Metric), IPC_7351 nominal, (Body size from: http://www.kemet.com/Lists/ProductCatalog/Attachments/253/KEM_TC101_STD.pdf), generated with kicad-footprint-generator")
@@
     (property "ki_keywords" "cap capacitor")
     (attr smd)
-    (fp_text reference "C4" (at 3.1538 -1.2474) (layer "F.Fab")
-        (effects (font (size 0.5 0.5) (thickness 0.125)))
+    (fp_text reference "C4" (at 0.0538 0.0526) (layer "F.Fab")
+        (effects (font (size 1 1) (thickness 0.15)))
     )
-    (fp_text value "330u" (at 3.0538 0.7026 90) (layer "F.Fab")
-        (effects (font (size 0.5 0.5) (thickness 0.125)))
+    (fp_text value "330u" (at 2.6538 0.0026 90) (layer "F.Fab")
+        (effects (font (size 1 1) (thickness 0.15)))
     )
     (fp_text user "${REFERENCE}" (at 0 0) (layer "F.Fab")
         (effects (font (size 0.88 0.88) (thickness 0.13)))
     )
-    (fp_line (start -2.635 -1.51) (end -2.635 1.51)
+    (fp_line (start -2.46 -1.51) (end -2.46 1.51)
       (stroke (width 0.12) (type solid)) (layer "F.SilkS"))
-    (fp_line (start -2.635 1.51) (end 1.75 1.51)
+    (fp_line (start -2.46 1.51) (end 1.75 1.51)
       (stroke (width 0.12) (type solid)) (layer "F.SilkS"))
-    (fp_line (start 1.75 -1.51) (end -2.635 -1.51)
+    (fp_line (start 1.75 -1.51) (end -2.46 -1.51)
       (stroke (width 0.12) (type solid)) (layer "F.SilkS"))
-    (fp_line (start -2.62 -1.65) (end 2.62 -1.65)
+    (fp_line (start -2.45 -1.65) (end 2.45 -1.65)
       (stroke (width 0.05) (type solid)) (layer "F.CrtYd"))
-    (fp_line (start -2.62 1.65) (end -2.62 -1.65)
+    (fp_line (start -2.45 1.65) (end -2.45 -1.65)
       (stroke (width 0.05) (type solid)) (layer "F.CrtYd"))
-    (fp_line (start 2.62 -1.65) (end 2.62 1.65)
+    (fp_line (start 2.45 -1.65) (end 2.45 1.65)
       (stroke (width 0.05) (type solid)) (layer "F.CrtYd"))
-    (fp_line (start 2.62 1.65) (end -2.62 1.65)
+    (fp_line (start 2.45 1.65) (end -2.45 1.65)
       (stroke (width 0.05) (type solid)) (layer "F.CrtYd"))
     (fp_line (start -1.75 -0.7) (end -1.75 1.4)
@@
     (fp_line (start 1.75 1.4) (end 1.75 -1.4)
       (stroke (width 0.1) (type solid)) (layer "F.Fab"))
-    (pad "1" smd roundrect (at -1.625 0) (size 1.5 2.35) (layers "F.Cu" "F.Paste" "F.Mask") (roundrect_rratio 0.1666673333)
+    (pad "1" smd roundrect (at -1.5375 0) (size 1.325 2.35) (layers "F.Cu" "F.Paste" "F.Mask") (roundrect_rratio 0.188679)
       (net 9 "Net-(BT1-+)") (pintype "passive"))
-    (pad "2" smd roundrect (at 1.625 0) (size 1.5 2.35) (layers "F.Cu" "F.Paste" "F.Mask") (roundrect_rratio 0.1666673333)
+    (pad "2" smd roundrect (at 1.5375 0) (size 1.325 2.35) (layers "F.Cu" "F.Paste" "F.Mask") (roundrect_rratio 0.188679)
       (net 1 "GND") (pintype "passive"))
     (model "${KICAD6_3DMODEL_DIR}/Capacitor_Tantalum_SMD.3dshapes/CP_EIA-3528-15_AVX-H.wrl"
@@
   (footprint "bwlr1e_prog:90055-AS" (layer "B.Cu")
     (at 162.687 103.0986 -90)
-    (property "Distributor Link" "https://www.digikey.com/en/products/detail/preci-dip/90055-AS/5451878")
     (property "Manufacturer" "Preci-Dip")
     (property "Part Number" "90055-AS")

Commit message: add usb-c receptacle
Parts:
- BT1: value 3.7v LiPo -> S2B-PH-SM4-TB
- J1: value DEBUG -> PinHeader_1x08_P2.54mm_Horizontal
- J2: value USB_C_Receptacle_USB2.0 -> U262-161N-4BVC11; footprint Teapot:USB_C_Receptacle_XKB_U262-16XN-4BVC11 -> bwlr1e_prog:USB_C_Receptacle_XKB_U262-16XN-4BVC11
- J3: value RESET -> PinHeader_1x02_P2.54mm_Horizontal
- J4: value BOOT -> PinHeader_1x02_P2.54mm_Horizontal
- SW1: value SW_DIP_x04 -> A6H-4101
- SW4: value BOOT -> TL3342F160QG
- SW5: value RESET -> TL3342F160QG
- TP1: value LIPO+ -> 90055-AS
- TP14: value BOOT -> 90055-AS
- TP2: value TXD2 -> 90055-AS
- TP3: value SWDIO -> 90055-AS
- TP4: value RXD2 -> 90055-AS
- TP5: value RST -> 90055-AS
- TP6: value SWCLK -> 90055-AS
- TP7: value GND -> 90055-AS
- TP8: value 3V3P -> 90055-AS
Changed lines of the file:
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@@
         (effects (font (size 1 1) (thickness 0.15)))
     )
-    (fp_text value "RESET" (at 0 3.75) (layer "F.Fab")
+    (fp_text value "TL3342F160QG" (at 0 3.75) (layer "F.Fab")
         (effects (font (size 1 1) (thickness 0.15)))
     )
@@
     (descr "LED SMD 0603 (1608 Metric), square (rectangular) end terminal, IPC_7351 nominal, (Body size source: http://www.tortai-tech.com/upload/download/2011102023233369053.pdf), generated with kicad-footprint-generator")
     (tags "LED")
-    (property "Part Number" "Orange 2V 25mA")
+    (property "Part Description" "Orange 2V 25mA")
     (property "Sheetfile" "bwlr1e-prog.kicad_sch")
     (property "Sheetname" "")
@@
         (effects (font (size 1 1) (thickness 0.15)))
     )
-    (fp_text value "DEBUG" (at 4.385 20.05) (layer "F.Fab")
+    (fp_text value "PinHeader_1x08_P2.54mm_Horizontal" (at 4.385 20.05) (layer "F.Fab")
         (effects (font (size 1 1) (thickness 0.15)))
     )
@@
         (effects (font (size 1 1) (thickness 0.15)))
     )
-    (fp_text value "RESET" (at 4.385 4.81) (layer "F.Fab")
+    (fp_text value "PinHeader_1x02_P2.54mm_Horizontal" (at 4.385 4.81) (layer "F.Fab")
         (effects (font (size 1 1) (thickness 0.15)))
     )
@@
         (effects (font (size 1 1) (thickness 0.15)))
     )
-    (fp_text value "BOOT" (at 0 3.75) (layer "F.Fab")
+    (fp_text value "TL3342F160QG" (at 0 3.75) (layer "F.Fab")
         (effects (font (size 1 1) (thickness 0.15)))
     )
@@
         (effects (font (size 1 1) (thickness 0.15)))
     )
-    (fp_text value "SW_DIP_x04" (at 0 2.7372 90) (layer "F.Fab")
+    (fp_text value "A6H-4101" (at 0 2.7372 90) (layer "F.Fab")
         (effects (font (size 0.5 0.5) (thickness 0.125)))
     )
@@
     )
   )
-  (footprint "Teapot:USB_C_Receptacle_XKB_U262-16XN-4BVC11" (layer "F.Cu")
+  (footprint "bwlr1e_prog:USB_C_Receptacle_XKB_U262-16XN-4BVC11" (layer "F.Cu")
     (at 146.556 139.895)
     (descr "USB Type C, right-angle, SMT, https://datasheet.lcsc.com/szlcsc/1811141824_XKB-Enterprise-U262-161N-4BVC11_C319148.pdf")
@@
     (property "ki_keywords" "usb universal serial bus type-C USB2.0")
     (attr smd)
-    (fp_text reference "J2" (at 0 0.005) (layer "F.Fab")
+    (fp_text reference "J2" (at 0.044 0.055) (layer "F.Fab")
         (effects (font (size 1 1) (thickness 0.15)))
     )
-    (fp_text value "USB_C_Receptacle_USB2.0" (at 0 4.935) (layer "F.Fab")
+    (fp_text value "U262-161N-4BVC11" (at 0 4.935) (layer "F.Fab")
         (effects (font (size 1 1) (thickness 0.15)))
     )
@@
     (pad "S1" thru_hole oval (at 4.32 1.075) (size 1 1.6) (drill oval 0.6 1.2) (layers "*.Cu" "*.Mask")
       (net 21 "unconnected-(J2-SHIELD-PadS1)") (pinfunction "SHIELD") (pintype "passive+no_connect"))
-    (model "${TEAPOT_3DMODEL_DIR}/u262-161n-4bvc11.stp"
+    (model "${KIPRJMOD}/library/3dmodels/u262-161n-4bvc11.stp"
       (offset (xyz 0 -3.65 1.7))
       (scale (xyz 1 1 1))
@@
         (effects (font (size 1 1) (thickness 0.15)))
     )
-    (fp_text value "BOOT" (at 4.385 4.81) (layer "F.Fab")
+    (fp_text value "PinHeader_1x02_P2.54mm_Horizontal" (at 4.385 4.81) (layer "F.Fab")
         (effects (font (size 1 1) (thickness 0.15)))
     )
@@
         (effects (font (size 1 1) (thickness 0.15)) (justify mirror))
     )
-    (fp_text value "3.7v LiPo" (at 0 -5.8 180) (layer "B.Fab")
+    (fp_text value "S2B-PH-SM4-TB" (at 0 -5.8 180) (layer "B.Fab")
         (effects (font (size 1 1) (thickness 0.15)) (justify mirror))
     )
@@
         (effects (font (size 0.5 0.5) (thickness 0.125)) (justify mirror))
     )
-    (fp_text value "GND" (at 0.0186 2.687 unlocked) (layer "F.Fab")
+    (fp_text value "90055-AS" (at 0.0186 2.687 unlocked) (layer "F.Fab")
         (effects (font (size 1 1) (thickness 0.15)))
     )
@@
         (effects (font (size 0.5 0.5) (thickness 0.125)) (justify mirror))
     )
-    (fp_text value "RXD2" (at -0.0018 4.087 unlocked) (layer "B.Fab")
+    (fp_text value "90055-AS" (at -0.0018 4.087 unlocked) (layer "B.Fab")
         (effects (font (size 1 1) (thickness 0.15)) (justify mirror))
     )
@@
         (effects (font (size 0.5 0.5) (thickness 0.125)) (justify mirror))
     )
-    (fp_text value "3V3P" (at 3.987 0.019 unlocked) (layer "B.Fab")
+    (fp_text value "90055-AS" (at 3.987 0.019 unlocked) (layer "B.Fab")
         (effects (font (size 1 1) (thickness 0.15)) (justify mirror))
     )
@@
         (effects (font (size 0.5 0.5) (thickness 0.125)) (justify mirror))
     )
-    (fp_text value "RST" (at 0 4.587 unlocked) (layer "B.Fab")
+    (fp_text value "90055-AS" (at 0 4.587 unlocked) (layer "B.Fab")
         (effects (font (size 1 1) (thickness 0.15)) (justify mirror))
     )
@@
         (effects (font (size 0.5 0.5) (thickness 0.125)) (justify mirror))
     )
-    (fp_text value "TXD2" (at 0 4.087 unlocked) (layer "B.Fab")
+    (fp_text value "90055-AS" (at 0 4.087 unlocked) (layer "B.Fab")
         (effects (font (size 1 1) (thickness 0.15)) (justify mirror))
     )
@@
         (effects (font (size 0.5 0.5) (thickness 0.125)) (justify mirror))
     )
-    (fp_text value "LIPO+" (at 0 3.887 unlocked) (layer "B.Fab")
+    (fp_text value "90055-AS" (at 0 3.887 unlocked) (layer "B.Fab")
         (effects (font (size 1 1) (thickness 0.15)) (justify mirror))
     )
@@
         (effects (font (size 0.5 0.5) (thickness 0.125)) (justify mirror))
     )
-    (fp_text value "SWCLK" (at 0.0498 3.587 unlocked) (layer "B.Fab")
+    (fp_text value "90055-AS" (at 0.0498 3.587 unlocked) (layer "B.Fab")
         (effects (font (size 1 1) (thickness 0.15)) (justify mirror))
     )
@@
         (effects (font (size 0.5 0.5) (thickness 0.125)) (justify mirror))
     )
-    (fp_text value "BOOT" (at 0.0158 -4.087 unlocked) (layer "B.Fab")
+    (fp_text value "90055-AS" (at 0.0158 -4.087 unlocked) (layer "B.Fab")
         (effects (font (size 1 1) (thickness 0.15)) (justify mirror))
     )
@@
         (effects (font (size 0.5 0.5) (thickness 0.125)) (justify mirror))
     )
-    (fp_text value "SWDIO" (at 0 3.587 unlocked) (layer "B.Fab")
+    (fp_text value "90055-AS" (at 0 3.587 unlocked) (layer "B.Fab")
         (effects (font (size 1 1) (thickness 0.15)) (justify mirror))
     )

Commit message: re-annotate
Parts:
- C4: renamed from C3; value 10nF -> 10n
- C5: value 100nF -> 100n
- renumbered C2 to C1, C4 to C2, C22 to C3, C23 to C6, C24 to C7, C26 to C8, C21 to C9, D4 to D1, H4 to H1, H1 to H2, H2 to H3, H3 to H4, J2 to J1, J1 to J2, R5 to R1, R1 to R2, R2 to R3, R14 to R5, R15 to R6, R17 to R7, R19 to R8, SW5 to SW2, SW4 to SW3, TP8 to TP1, TP1 to TP2, TP2 to TP3, TP14 to TP5, TP5 to TP6, TP6 to TP7, TP3 to TP8, TP7 to TP9, U7 to U1, U1 to U2, U8 to U3, U6 to U4

Commit message: update footprint library
Parts:
- G***: footprint bwlr1e:TeapotLogo4mm -> bwlr1e_prog:TeapotLogo4mm
- REF**: footprint bwlr1e:EdgeCut_BWLR1E -> bwlr1e_prog:EdgeCut_BWLR1E
