File: hardware/main/kicad/bwlr1e.kicad_pcb (KiCad board)
At the start: 2 copper layers, 36.8 x 90.9 mm, 65 parts, among them J1 Qwiic, Q1 AO3407A, Q2 DMG1012UW, SW3 RESET, SW4 BOOT, U1 BME688, U2 RAK3172-T, U3 AEM10941, U4 XC6215

Commit message: change csrc aem10941 to 10uf
Parts:
- C6: value 150u -> 10u; footprint Capacitor_SMD:C_1210_3225Metric -> Capacitor_SMD:C_0603_1608Metric
- moved C6 1.18 mm to (147.8, 105.7)
Other:
- board text added: "3V7 LIPO"
- board text added: "Revision 5"
- board text removed: "3.7v LiPo"
- board text removed: "Revision 4"
Changed lines of the file:
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@@
   (title_block
     (title "Teapotlabs BWLR1E")
-    (date "2023-08-12")
-    (rev "4")
+    (date "2023-09-26")
+    (rev "5")
     (company "Teapot Laboratories")
   )
@@
     )
   )
-  (footprint "Capacitor_SMD:C_1210_3225Metric" (layer "F.Cu")
-    (at 148.8 105 90)
-    (descr "Capacitor SMD 1210 (3225 Metric), square (rectangular) end terminal, IPC_7351 nominal, (Body size source: IPC-SM-782 page 76, https://www.pcb-3d.com/wordpress/wp-content/uploads/ipc-sm-782a_amendment_1_and_2.pdf), generated with kicad-footprint-generator")
+  (footprint "Capacitor_SMD:C_0603_1608Metric" (layer "F.Cu")
+    (at 147.828 105.664 90)
+    (descr "Capacitor SMD 0603 (1608 Metric), square (rectangular) end terminal, IPC_7351 nominal, (Body size source: IPC-SM-782 page 76, https://www.pcb-3d.com/wordpress/wp-content/uploads/ipc-sm-782a_amendment_1_and_2.pdf), generated with kicad-footprint-generator")
     (tags "capacitor")
-    (property "Part Description" "Ceramic Capacitor 150uF 20% 6.3V X5R")
+    (property "Distributor" "")
+    (property "Distributor Link" "")
+    (property "Distributor Part Number" "")
+    (property "Manufacturer" "")
+    (property "Manufacturer Part Number" "")
+    (property "Part Description" "Ceramic Capacitor 10uF 10% 10V X5R")
     (property "Sheetfile" "bwlr1e.kicad_sch")
     (property "Sheetname" "")
@@
     (property "ki_keywords" "capacitor cap")
     (attr smd)
-    (fp_text reference "C6" (at 1.749 2.203 180) (layer "F.SilkS")
+    (fp_text reference "C6" (at 1.27 1.778 180) (layer "F.SilkS")
         (effects (font (size 0.5 0.5) (thickness 0.125)))
     )
-    (fp_text value "150u" (at -0.029 2.076 90) (layer "F.Fab")
-        (effects (font (size 0.5 0.5) (thickness 0.125)))
+    (fp_text value "10u" (at 0 1.43 90) (layer "F.Fab")
+        (effects (font (size 1 1) (thickness 0.15)))
     )
     (fp_text user "${REFERENCE}" (at 0 0 90) (layer "F.Fab")
-        (effects (font (size 0.8 0.8) (thickness 0.12)))
+        (effects (font (size 0.4 0.4) (thickness 0.06)))
     )
-    (fp_line (start -0.711252 -1.36) (end 0.711252 -1.36)
+    (fp_line (start -0.14058 -0.51) (end 0.14058 -0.51)
       (stroke (width 0.12) (type solid)) (layer "F.SilkS"))
-    (fp_line (start -0.711252 1.36) (end 0.711252 1.36)
+    (fp_line (start -0.14058 0.51) (end 0.14058 0.51)
       (stroke (width 0.12) (type solid)) (layer "F.SilkS"))
-    (fp_line (start -2.3 -1.6) (end 2.3 -1.6)
+    (fp_line (start -1.48 -0.73) (end 1.48 -0.73)
       (stroke (width 0.05) (type solid)) (layer "F.CrtYd"))
-    (fp_line (start -2.3 1.6) (end -2.3 -1.6)
+    (fp_line (start -1.48 0.73) (end -1.48 -0.73)
       (stroke (width 0.05) (type solid)) (layer "F.CrtYd"))
-    (fp_line (start 2.3 -1.6) (end 2.3 1.6)
+    (fp_line (start 1.48 -0.73) (end 1.48 0.73)
       (stroke (width 0.05) (type solid)) (layer "F.CrtYd"))
-    (fp_line (start 2.3 1.6) (end -2.3 1.6)
+    (fp_line (start 1.48 0.73) (end -1.48 0.73)
       (stroke (width 0.05) (type solid)) (layer "F.CrtYd"))
-    (fp_line (start -1.6 -1.25) (end 1.6 -1.25)
+    (fp_line (start -0.8 -0.4) (end 0.8 -0.4)
       (stroke (width 0.1) (type solid)) (layer "F.Fab"))
-    (fp_line (start -1.6 1.25) (end -1.6 -1.25)
+    (fp_line (start -0.8 0.4) (end -0.8 -0.4)
       (stroke (width 0.1) (type solid)) (layer "F.Fab"))
-    (fp_line (start 1.6 -1.25) (end 1.6 1.25)
+    (fp_line (start 0.8 -0.4) (end 0.8 0.4)
       (stroke (width 0.1) (type solid)) (layer "F.Fab"))
-    (fp_line (start 1.6 1.25) (end -1.6 1.25)
+    (fp_line (start 0.8 0.4) (end -0.8 0.4)
       (stroke (width 0.1) (type solid)) (layer "F.Fab"))
-    (pad "1" smd roundrect (at -1.475 0 90) (size 1.15 2.7) (layers "F.Cu" "F.Paste" "F.Mask") (roundrect_rratio 0.2173913043)
+    (pad "1" smd roundrect (at -0.775 0 90) (size 0.9 0.95) (layers "F.Cu" "F.Paste" "F.Mask") (roundrect_rratio 0.25)
       (net 11 "Net-(U3-BUFSRC)") (pintype "passive"))
-    (pad "2" smd roundrect (at 1.475 0 90) (size 1.15 2.7) (layers "F.Cu" "F.Paste" "F.Mask") (roundrect_rratio 0.2173913043)
+    (pad "2" smd roundrect (at 0.775 0 90) (size 0.9 0.95) (layers "F.Cu" "F.Paste" "F.Mask") (roundrect_rratio 0.25)
       (net 2 "GND") (pintype "passive"))
-    (model "${KICAD6_3DMODEL_DIR}/Capacitor_SMD.3dshapes/C_1210_3225Metric.wrl"
+    (model "${KICAD6_3DMODEL_DIR}/Capacitor_SMD.3dshapes/C_0603_1608Metric.wrl"
       (offset (xyz 0 0 0))
       (scale (xyz 1 1 1))
@@
     (property "ki_keywords" "battery cell")
     (attr smd)
-    (fp_text reference "BT1" (at -3.206 -5.842 180) (layer "B.SilkS")
+    (fp_text reference "BT1" (at -5.492 3.937 -90) (layer "B.SilkS")
         (effects (font (size 1 1) (thickness 0.15)) (justify mirror))
     )
@@
     (pad "2" smd roundrect (at 1 2.85) (size 1 3.5) (layers "B.Cu" "B.Paste" "B.Mask") (roundrect_rratio 0.25)
       (net 2 "GND") (pinfunction "-") (pintype "passive"))
-    (pad "MP" smd roundrect (at -3.35 -2.9) (size 1.5 3.4) (layers "B.Cu" "B.Paste" "B.Mask") (roundrect_rratio 0.166667))
-    (pad "MP" smd roundrect (at 3.35 -2.9) (size 1.5 3.4) (layers "B.Cu" "B.Paste" "B.Mask") (roundrect_rratio 0.166667))
+    (pad "MP" smd roundrect (at -3.35 -2.9) (size 1.5 3.4) (layers "B.Cu" "B.Paste" "B.Mask") (roundrect_rratio 0.1666673333))
+    (pad "MP" smd roundrect (at 3.35 -2.9) (size 1.5 3.4) (layers "B.Cu" "B.Paste" "B.Mask") (roundrect_rratio 0.1666673333))
     (model "${KIPRJMOD}/library/3dmodels/S2B-PH-SM4-TB.STEP"
       (offset (xyz 0 -4.4 0))
@@
     (pad "4" smd roundrect (at 1.5 2 90) (size 0.6 1.55) (layers "B.Cu" "B.Paste" "B.Mask") (roundrect_rratio 0.25)
       (net 14 "/SCL") (pinfunction "Pin_4") (pintype "passive"))
-    (pad "MP" smd roundrect (at -2.8 -1.875 90) (size 1.2 1.8) (layers "B.Cu" "B.Paste" "B.Mask") (roundrect_rratio 0.208333))
-    (pad "MP" smd roundrect (at 2.8 -1.875 90) (size 1.2 1.8) (layers "B.Cu" "B.Paste" "B.Mask") (roundrect_rratio 0.208333))
+    (pad "MP" smd roundrect (at -2.8 -1.875 90) (size 1.2 1.8) (layers "B.Cu" "B.Paste" "B.Mask") (roundrect_rratio 0.2083333333))
+    (pad "MP" smd roundrect (at 2.8 -1.875 90) (size 1.2 1.8) (layers "B.Cu" "B.Paste" "B.Mask") (roundrect_rratio 0.2083333333))
     (model "${KIPRJMOD}/library/3dmodels/SM04B-SRSS-TB.STEP"
       (offset (xyz 0 1.3 -0.3))
@@
     (effects (font (size 0.5 0.5) (thickness 0.125)) (justify left bottom mirror))
   )
-  (gr_text "Revision 4" (at 161.925 142.367) (layer "B.SilkS" knockout)
+  (gr_text "Revision 5" (at 161.925 142.367) (layer "B.SilkS" knockout)
     (effects (font (size 0.8 0.8) (thickness 0.2) bold) (justify left bottom mirror))
   )
@@
     (effects (font (size 1.5 1.5) (thickness 0.3)) (justify mirror))
   )
-  (gr_text "3.7v LiPo" (at 160.909 127) (layer "B.SilkS")
-    (effects (font (size 0.5 0.5) (thickness 0.125)) (justify mirror))
+  (gr_text "3V7 LIPO" (at 158.242 126.238 180) (layer "B.SilkS" knockout)
+    (effects (font (size 1 1) (thickness 0.15)) (justify mirror))
   )
   (gr_text "SOLAR HARVESTER" (at 131.6228 114.046) (layer "F.SilkS" knockout)
@@
   (segment (start 132.45 74.7125) (end 132.4375 74.7) (width 0.5) (layer "F.Cu") (net 10))
   (segment (start 132.4375 73.0875) (end 132.4375 76.3016) (width 1) (layer "F.Cu") (net 10))
+  (segment (start 147.333 106.439) (end 146.365 105.471) (width 0.5) (layer "F.Cu") (net 11))
   (segment (start 144.198 108.45) (end 144.198 107.167) (width 0.25) (layer "F.Cu") (net 11))
   (segment (start 144.198 107.167) (end 146.365 105) (width 0.25) (layer "F.Cu") (net 11))
-  (segment (start 147.84 106.475) (end 146.365 105) (width 1) (layer "F.Cu") (net 11))
-  (segment (start 148.8 106.475) (end 147.84 106.475) (width 1) (layer "F.Cu") (net 11))
+  (segment (start 146.365 105.471) (end 146.365 105) (width 0.5) (layer "F.Cu") (net 11))
+  (segment (start 147.3135 106.426) (end 146.8185 106.426) (width 0.5) (layer "F.Cu") (net 11))
+  (segment (start 146.8055 106.426) (end 146.3105 106.426) (width 0.5) (layer "F.Cu") (net 11))
   (segment (start 141.9225 107.6325) (end 141.3 107.01) (width 0.25) (layer "F.Cu") (net 12))
   (segment (start 141.3 107.01) (end 141.3 105.9625) (width 0.25) (layer "F.Cu") (net 12))
