File: hardware/programmer/kicad/bwlr1e-prog.kicad_sch (KiCad schematic)
At the start: 46 parts, among them J1 U262-161N-4BVC11, J2 PinHeader_1x08_P2.54mm_Horizo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, J3 PinHeader_1x02_P2.54mm_Horizo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, J4 PinHeader_1x02_P2.54mm_Horizo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, Q1 AO3407A, SW1 A6H-4101, SW2 TL3342F160QG, SW3 TL3342F160QG, U1 MCP73831T-2ACI/OT, U2 USBLC6-2P6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

Commit message: update component value
Parts:
- C1, C2: Manufacturer KYOCERA AVX -> KEMET; Part Number TPSB476K010R0350 -> T520B337M006ATE040
Changed lines of the file:
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@@
       (effects (font (size 1.27 1.27)) hide)
     )
-    (property "Datasheet" "https://datasheets.kyocera-avx.com/TPS.pdf" (at 53.34 175.895 0)
+    (property "Datasheet" "" (at 53.34 175.895 0)
       (effects (font (size 1.27 1.27)) hide)
     )
-    (property "Manufacturer" "KYOCERA AVX" (at 53.34 175.895 0)
+    (property "Manufacturer" "KEMET" (at 53.34 175.895 0)
       (effects (font (size 1.27 1.27)) hide)
     )
-    (property "Part Number" "TPSB476K010R0350" (at 53.34 175.895 0)
+    (property "Part Number" "T520B337M006ATE040" (at 53.34 175.895 0)
       (effects (font (size 1.27 1.27)) hide)
     )
@@
       (effects (font (size 1.27 1.27)) hide)
     )
-    (property "Datasheet" "https://datasheets.kyocera-avx.com/TPS.pdf" (at 41.91 175.895 0)
+    (property "Datasheet" "" (at 41.91 175.895 0)
       (effects (font (size 1.27 1.27)) hide)
     )
-    (property "Manufacturer" "KYOCERA AVX" (at 41.91 175.895 0)
+    (property "Manufacturer" "KEMET" (at 41.91 175.895 0)
       (effects (font (size 1.27 1.27)) hide)
     )
-    (property "Part Number" "TPSB476K010R0350" (at 41.91 175.895 0)
+    (property "Part Number" "T520B337M006ATE040" (at 41.91 175.895 0)
       (effects (font (size 1.27 1.27)) hide)
     )

Commit message: clean-up
Parts:
- FB1: symbol Penguino-STM32WL-LoRa-E5-rescue:Ferrite_Bead-Device -> Device:FerriteBead
Changed lines of the file:
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@@
     )
   )
-  (symbol (lib_id "Penguino-STM32WL-LoRa-E5-rescue:Ferrite_Bead-Device") (at 89.535 29.21 90) (unit 1)
+  (symbol (lib_id "Device:FerriteBead") (at 89.535 29.21 90) (unit 1)
     (in_bom yes) (on_board yes) (dnp no)
     (property "Reference" "FB1" (at 86.36 27.94 90)
@@
       (effects (font (size 1.27 1.27)) hide)
     )
+    (property "Part Description" "" (at 89.535 29.21 0)
+      (effects (font (size 1.27 1.27)) hide)
+    )
+    (property "Manufacturer Part Number" "" (at 89.535 29.21 0)
+      (effects (font (size 1.27 1.27)) hide)
+    )
+    (property "Distributor" "" (at 89.535 29.21 0)
+      (effects (font (size 1.27 1.27)) hide)
+    )
+    (property "Distributor Part Number" "" (at 89.535 29.21 0)
+      (effects (font (size 1.27 1.27)) hide)
+    )
+    (property "Distributor Link" "" (at 89.535 29.21 0)
+      (effects (font (size 1.27 1.27)) hide)
+    )
